File: vkc-keyboard/vitter-kb.kicad_pcb (KiCad board)
At the start: 2 copper layers, 70 parts, among them SW1 SW_SPST, SW10 SW_SPST, SW11 SW_SPST, SW12 SW_SPST, SW13 SW_SPST, SW14 SW_SPST, SW15 SW_SPST, SW16 SW_SPST, SW17 SW_SPST, SW18 SW_SPST, SW19 SW_SPST, SW2 SW_SPST, SW20 SW_SPST, SW21 SW_SPST, SW22 SW_SPST, SW23 SW_SPST, SW24 SW_SPST, SW25 SW_SPST, SW26 SW_SPST, SW27 SW_SPST, SW28 SW_SPST, SW29 SW_SPST, SW3 SW_SPST, SW30 SW_SPST, SW31 SW_SPST, SW32 SW_SPST, SW33 SW_SPST, SW34 SW_SPST, SW35 SW_SPST, SW4 SW_SPST, SW5 SW_SPST, SW6 SW_SPST, SW7 SW_SPST, SW8 SW_SPST, SW9 SW_SPST

Commit message: bingo
Parts:
- removed D1, D10, D11, D12, D13, D14, D15, D16, D17, D18, D19, D2, D20, D21, D22, D23, D24, D25, D26, D27, D28, D29, D3, D30, D31, D32, D33, D34, D35, D4, D5, D6, D7, D8, D9: 1N4148, vitter-kb:Diode-dual
- added SW36: SW_SPST, vitter-kb:Kailh_socket_PG1350_reversible, F.Cu at (36.6, 47.6)
- added SW37: SW_SPST, vitter-kb:Kailh_socket_PG1350_reversible, F.Cu at (54.6, 45.6)
- added SW38: SW_SPST, vitter-kb:Kailh_socket_PG1350_reversible, F.Cu at (72.6, 42.6)
- added SW39: SW_SPST, vitter-kb:Kailh_socket_PG1350_reversible, F.Cu at (90.6, 41.6)
- moved SW7 12.0 mm to (144.6, 69.7)
- moved SW14 12.0 mm to (144.6, 86.7)
- moved SW21 12.0 mm to (144.6, 103.7)
- moved SW28 12.0 mm to (144.6, 120.7)
- moved SW35 12.0 mm to (144.6, 137.7)
- moved SW12 11.0 mm to (108.6, 80.7)
- moved SW19 11.0 mm to (108.6, 97.7)
- moved SW26 11.0 mm to (108.6, 114.7)
- moved SW33 11.0 mm to (108.6, 131.7)
- moved SW5 11.0 mm to (108.6, 63.6)
- moved SW6 8.00 mm to (126.6, 65.7)
- moved SW13 8.00 mm to (126.6, 82.7)
- moved SW20 8.00 mm to (126.6, 99.7)
- moved SW27 8.00 mm to (126.6, 116.7)
- moved SW34 8.00 mm to (126.6, 133.7)
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
Commit message: route
Parts:
- added D1: 1N4148, vitter-kb:Diode-SOD-123-FB, F.Cu at (36.5, 59.9)
- added D10: 1N4148, vitter-kb:Diode-SOD-123-FB, F.Cu at (72.7, 71.8)
- added D11: 1N4148, vitter-kb:Diode-SOD-123-FB, F.Cu at (90.8, 71.0)
- added D12: 1N4148, vitter-kb:Diode-SOD-123-FB, F.Cu at (108.6, 76.0)
- added D13: 1N4148, vitter-kb:Diode-SOD-123-FB, F.Cu at (126.5, 78.0)
- added D14: 1N4148, vitter-kb:Diode-SOD-123-FB, F.Cu at (144.8, 82.0)
- added D15: 1N4148, vitter-kb:Diode-SOD-123-FB, F.Cu at (36.5, 94.0)
- added D16: 1N4148, vitter-kb:Diode-SOD-123-FB, F.Cu at (54.5, 92.0)
- added D17: 1N4148, vitter-kb:Diode-SOD-123-FB, F.Cu at (72.5, 89.0)
- added D18: 1N4148, vitter-kb:Diode-SOD-123-FB, F.Cu at (90.6, 87.9)
- added D19: 1N4148, vitter-kb:Diode-SOD-123-FB, F.Cu at (108.5, 92.9)
- added D2: 1N4148, vitter-kb:Diode-SOD-123-FB, F.Cu at (54.4, 58.0)
- added D20: 1N4148, vitter-kb:Diode-SOD-123-FB, F.Cu at (126.5, 95.0)
- added D21: 1N4148, vitter-kb:Diode-SOD-123-FB, F.Cu at (144.6, 99.0)
- added D22: 1N4148, vitter-kb:Diode-SOD-123-FB, F.Cu at (36.5, 111.0)
- added D23: 1N4148, vitter-kb:Diode-SOD-123-FB, F.Cu at (54.5, 109.0)
- added D24: 1N4148, vitter-kb:Diode-SOD-123-FB, F.Cu at (72.6, 105.8)
- added D25: 1N4148, vitter-kb:Diode-SOD-123-FB, F.Cu at (90.5, 105.0)
- added D26: 1N4148, vitter-kb:Diode-SOD-123-FB, F.Cu at (108.5, 109.9)
- added D27: 1N4148, vitter-kb:Diode-SOD-123-FB, F.Cu at (126.5, 112.0)
- added D28: 1N4148, vitter-kb:Diode-SOD-123-FB, F.Cu at (144.6, 116.1)
- added D29: 1N4148, vitter-kb:Diode-SOD-123-FB, F.Cu at (36.6, 127.9)
- added D3: 1N4148, vitter-kb:Diode-SOD-123-FB, F.Cu at (72.6, 55.0)
- added D30: 1N4148, vitter-kb:Diode-SOD-123-FB, F.Cu at (54.6, 126.0)
- added D31: 1N4148, vitter-kb:Diode-SOD-123-FB, F.Cu at (72.5, 123.0)
- added D32: 1N4148, vitter-kb:Diode-SOD-123-FB, F.Cu at (90.6, 122.0)
- added D33: 1N4148, vitter-kb:Diode-SOD-123-FB, F.Cu at (108.6, 127.0)
- added D34: 1N4148, vitter-kb:Diode-SOD-123-FB, F.Cu at (126.5, 129.0)
- added D35: 1N4148, vitter-kb:Diode-SOD-123-FB, F.Cu at (144.6, 133.1)
- added D36: 1N4148, vitter-kb:Diode-SOD-123-FB, F.Cu at (36.6, 42.8)
- added D37: 1N4148, vitter-kb:Diode-SOD-123-FB, F.Cu at (54.5, 40.8)
- added D38: 1N4148, vitter-kb:Diode-SOD-123-FB, F.Cu at (72.3, 37.8)
- added D39: 1N4148, vitter-kb:Diode-SOD-123-FB, F.Cu at (90.3, 37.0)
- added D4: 1N4148, vitter-kb:Diode-SOD-123-FB, F.Cu at (90.5, 53.8)
- added D5: 1N4148, vitter-kb:Diode-SOD-123-FB, F.Cu at (108.6, 59.0)
- added D6: 1N4148, vitter-kb:Diode-SOD-123-FB, F.Cu at (126.6, 61.0)
- added D7: 1N4148, vitter-kb:Diode-SOD-123-FB, F.Cu at (144.6, 64.8)
- added D8: 1N4148, vitter-kb:Diode-SOD-123-FB, B.Cu at (36.6, 77.0)
- added D9: 1N4148, vitter-kb:Diode-SOD-123-FB, B.Cu at (54.6, 74.6)
- added H1: MountingHole, MountingHole:MountingHole_2.2mm_M2, F.Cu at (134.1, 56.0)
- added H2: MountingHole, MountingHole:MountingHole_2.2mm_M2, F.Cu at (101.4, 40.9)
- added H4: MountingHole, MountingHole:MountingHole_2.2mm_M2, F.Cu at (141.7, 66.2)
- added J1: TRRS, vitter-kb:TRRS-PJ-320A, F.Cu at (150.9, 57.6)
- added J2: TRRS, vitter-kb:TRRS-PJ-320A, B.Cu at (150.9, 53.0)
- added U1: ProMicro_r, vitter-kb:ProMicro_v2, B.Cu at (121.6, 39.9)
Routing:
- net /col1: track 0.00 -> 328.6 mm, vias 0 -> 8
- net /col2: track 0.00 -> 305.0 mm, vias 0 -> 8
- net /col3: track 0.00 -> 284.0 mm, vias 0 -> 8
- net /row5: track 0.00 -> 248.6 mm, vias 0 -> 8
- net /row4: track 0.00 -> 232.7 mm, vias 0 -> 8
- net /col7: track 0.00 -> 229.1 mm, vias 0 -> 5
- net /col6: track 0.00 -> 220.3 mm, vias 0 -> 7
- net /col4: track 0.00 -> 219.4 mm, vias 0 -> 7
- net /row3: track 0.00 -> 218.1 mm, vias 0 -> 8
- net /row1: track 0.00 -> 216.6 mm, vias 0 -> 7
- net /col5: track 0.00 -> 216.1 mm, vias 0 -> 7
- net /row2: track 0.00 -> 209.2 mm, vias 0 -> 8
- net /row0: track 0.00 -> 121.8 mm, vias 0 -> 5
- net +3.3V: track 0.00 -> 34.7 mm
- net rx: track 0.00 -> 27.5 mm
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Other:
- board outline added: 128.5 x 117.6 mm
