File: vkc-keyboard/vitter-kb.kicad_pcb (KiCad board)
At the start: 2 copper layers, 128.5 x 117.6 mm, 84 parts, among them J1 TRRS, J2 TRRS, SW1 SW_SPST, SW10 SW_SPST, SW11 SW_SPST, SW12 SW_SPST, SW13 SW_SPST, SW14 SW_SPST, SW15 SW_SPST, SW16 SW_SPST, SW17 SW_SPST, SW18 SW_SPST, SW19 SW_SPST, SW2 SW_SPST, SW20 SW_SPST, SW21 SW_SPST, SW22 SW_SPST, SW23 SW_SPST, SW24 SW_SPST, SW25 SW_SPST, SW26 SW_SPST, SW27 SW_SPST, SW28 SW_SPST, SW29 SW_SPST, SW3 SW_SPST, SW30 SW_SPST, SW31 SW_SPST, SW32 SW_SPST, SW33 SW_SPST, SW34 SW_SPST, SW35 SW_SPST, SW36 SW_SPST, SW37 SW_SPST, SW38 SW_SPST, SW39 SW_SPST, SW4 SW_SPST, SW5 SW_SPST, SW6 SW_SPST, SW7 SW_SPST, SW8 SW_SPST, SW9 SW_SPST, U1 ProMicro_r

Commit message: ryg venstre kolone og tre højre 2mm ned
Parts:
- moved SW5 2.00 mm to (108.6, 65.7)
- moved D1 2.00 mm to (36.5, 61.9)
- moved D12 2.00 mm to (108.6, 78.0)
- moved D13 2.00 mm to (126.5, 80.0)
- moved D14 2.00 mm to (144.8, 84.0)
- moved D15 2.00 mm to (36.5, 96.0)
- moved D19 2.00 mm to (108.5, 94.9)
- moved D20 2.00 mm to (126.5, 97.0)
- moved D21 2.00 mm to (144.6, 101.0)
- moved D22 2.00 mm to (36.5, 113.0)
- moved D26 2.00 mm to (108.5, 111.9)
- moved D27 2.00 mm to (126.5, 114.0)
- moved D28 2.00 mm to (144.6, 118.1)
- moved D29 2.00 mm to (36.6, 129.9)
- moved D33 2.00 mm to (108.6, 129.0)
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Routing:
- net /col1: track 328.6 -> 334.5 mm
- net Net-(D15-A): track 24.6 -> 19.8 mm
- net Net-(D6-A): track 23.9 -> 27.9 mm
- net Net-(D5-A): track 23.9 -> 27.9 mm
- net Net-(D36-A): track 24.3 -> 28.3 mm
- net /col5: track 216.1 -> 218.5 mm
- net /col7: track 229.1 -> 231.1 mm
- net /col6: track 220.3 -> 222.3 mm
- net /row1: track 216.6 -> 218.5 mm
- net /row2: track 209.2 -> 210.1 mm
- net Net-(D29-A): track 24.1 -> 23.5 mm
- net /row5: track 248.6 -> 249.1 mm
Other:
- board size 128.5 x 117.6 mm -> 128.5 x 119.6 mm
